Commit message: updated codes, arucos, words

File: src/puzzlebot_gazebo/urdf/parameters.xacro (robot description, xacro)
@@ -6,5 +6,4 @@
 <xacro:property name="chassisY" value="0.16"/>
 <xacro:property name="chassisZ" value="0.06"/>
-<!-- <xacro:property name="chassisMass" value="0.710"/> -->
 <xacro:property name="chassisMass" value="1.219"/>
 <xacro:property name="casterRadius" value="0.0065"/>
@@ -24,3 +23,4 @@
 <xacro:property name="mesh_camera"  value="$(find puzzlebot_gazebo)/meshes/camera.stl" />
 <xacro:property name="mesh_lidar"  value="$(find puzzlebot_gazebo)/meshes/lidar.stl" />
+<xacro:property name="mesh_gripper" value="$(find puzzlebot_gazebo)/meshes/GripperSTL.stl" />
 </robot>

File: src/puzzlebot_gazebo/urdf/puzzlebot.xacro (robot description, xacro)
@@ -186,4 +186,31 @@
 		</inertial>]]>
     </link>
+	<!-- GRIPPER -->
+	 <link name="gripper">
+		    <inertial>
+		    	    <origin rpy="0 0 0" xyz="0 0 0"/>
+		          <mass value="0.007"/>
+		          <inertia ixx="0.166667" ixy="0" ixz="0" iyy="0.166667" iyz="0" izz="0.166667"/>
+		          <!-- ad camera inertia -->
+		    </inertial>
+			<collision name="collision_chassis">
+		    	    <origin rpy="0 0 0" xyz="0 0 0"/>
+		          <geometry>
+		               <box size="0.05 0.01 0.06" />
+		          </geometry>
+		    </collision>
+		    <visual>
+		    	    <!-- box only
+		    	    <origin rpy="$0 0 ${PI/2}" xyz="0 0 0"/>
+		          <geometry>
+		          	<box size="0.05 0.01 0.06" />
+		          </geometry>-->
+		         <!-- with mesh-->
+		          <origin rpy="${PI/1.8} 0.07 ${-PI/2.25}" xyz="0.06 0.03 -0.06"/>
+		          <geometry>
+		          	<mesh filename="file://${mesh_gripper}" scale="0.0009 0.0009 0.0009" />
+		          </geometry>
+		    </visual>
+  </link>
 	<!-- JOINTS  -->
 	<joint name="base_to_right_w" type="continuous">
@@ -220,4 +247,9 @@
         <origin xyz="0.05 0 0.115" rpy="0 0 ${PI}"/>
     </joint>
+<joint name="gripper_to_base" type="fixed">
+	  <parent link="chassis" />
+	  <child link="gripper" />
+	  <origin xyz="0.149 0.031 .038" rpy= "0.0 0.24 0.0" />
+  </joint>
 	<!-- TRANSMISSIONS (For a more complex model and it represents actuator attributes) -->
 	<transmission name="right_wheel_trans">
